File: 0003-Stm32PcbDesign/Noin-main/Noinminiv3/Noinminiv3.kicad_sch (KiCad schematic)
At the start: 33 parts, among them J1 USB_C_Receptacle_USB2.0_16P, J2 PINHD_1x10_Female, J4 PINHD_1x5_Male, J5 PINHD_1x10_Female, SW1 Push_Button, U1 AP2112K-3.3TRG1, U2 ATSAMD21E16B-M

Commit message: added library
Parts:
- C1, C10, C11, C2, C3, C4, C5, C6, C7, C8, C9: symbol PCM_4ms_Capacitor:1uF_0603_25V -> all-comps:1uF_0603_25V
- D1: symbol Diode:MBR1020VL -> all-comps:MBR1020VL
- D2: symbol PCM_Diode_TVS_AKL:USBLC6-2SC6 -> all-comps:USBLC6-2SC6
- F1: symbol Device:Fuse_Small -> all-comps:Fuse_Small
- J1: symbol Connector:USB_C_Receptacle_USB2.0_16P -> all-comps:USB_C_Receptacle_USB2.0_16P
- J2, J5: symbol PCM_SL_Pin_Headers:PINHD_1x10_Female -> all-comps:PINHD_1x10_Female
- J4: symbol PCM_SL_Pin_Headers:PINHD_1x5_Male -> all-comps:PINHD_1x5_Male
- LED1, LED2: symbol PCM_LED_AKL:LED_1.8mm_SMD_Red -> all-comps:LED_1.8mm_SMD_Red
- R1, R2, R3, R4, R5, R6, R7, R8, R9: symbol PCM_4ms_Resistor:10k_0402 -> all-comps:10k_0402
- R10: symbol EE_RESISTORS:0402WGF1001TCE -> all-comps:0402WGF1001TCE
- SW1: symbol PCM_SL_Devices:Push_Button -> all-comps:Push_Button
- U1: symbol PCM_Voltage_Regulator_AKL:AP2112K-3.3TRG1 -> all-comps:AP2112K-3.3TRG1
- U2: symbol MCU_Microchip_SAMD:ATSAMD21E16B-M -> all-comps:ATSAMD21E16B-M
Changed lines of the file:
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@@
 			"AAAAAAAAAAAAAAAAAAAAAAAAAAAAAAAAAAAAAAAAAAAAAAAAAAAAAAAAAAAAAAAAAAAAAAAAAAAA"
 			"AAAAAAAAAAAAAAAAAAAAAAAAAAAAAAAAAAAAAAAAAAAAAAAAAAAAAAAAAAAAAAAAAAAAAAAAAAAA"
+			"AAAAAAAAAAAAAAAAAAAAAAAAAAAAAAAAAAAAAAAAAAAAAAAAAAAAAAAAAAAAAAAAAAAAAAAAAAAA"
+			"AAAAAAAAAAAAAAAAAAAAAAAAAAAAAAAAAAAAAAAAAAAAAAAAAAAAAAAAAAAAAAAAAAAAAAAAAAAA"
+			"AAAAAAAAAAAAAAAAAAAAAAAAAAAAAAAAAAAAAAAAAAAAAAAAAAAAAAAAAAAAAAAAAAAAAAAAAAAA"
+			"AAAAAAAAAAAAAAAAAAAAAAAAAAAAAAAAAAAAAAAAAAAAAAAAAAAAAAAAAAAAAAAAAAAAAAAAAAAA"
+			"AAAAAAAAAAAAAAAAAAAAAAAAAAAAAAAAAAAAAAAAAAAAAAAAAAAAAAAAAAAAAAAAAAAAAAAAAAAA"
+			"AAAAAAAAAAAAAAAAAAAAAAAAAAAAAAAAAAAAAAAAAAAAAAAAAAAAAAAAAAAAAAAAAAAAAAAAAAAA"
+			"AAAAAAAAAAAAAAAAAAAAAAAAAAAAAAAAAAAAAAAAAAAAAAAAAAAAAAAAAAAAAAAAAAAAAAAAAAAA"
+			"AAAAAAAAAAAAAAAAAAAAAAAAAAAAAAAAAAAAAAAAAAAAAAAAAAAAAAAAAAAAAAAAAAAAAAAAAAAA"
+			"AAAAAAAAAAAAAAAAAAAAAAAAAAAAAAAAAAAAAAAAAAAAAAAAAAAAAAAAAAAAAAAAAAAAAAAAAAAA"
+			"AAAAAAAAAAAAAAAAAAAAAAAAAAAAAAAAAAAAAAAAAAAAAAAAAAAAAAAAAAAAAAAAAAAAAAAAAAAA"
+			"AAAAAAAAAAAAAAAAAAAAAAAAAAAAAAAAAAAAAAAAAAAAAAAAAAAAAAAAAAAAAAAAAAAAAAAAAAAA"
+			"AAAAAAAAAAAAAAAAAAAAAAAAAAAAAAAAAAAAAAAAAAAAAAAAAAAAAAAAAAAAAAAAAAAAAAAAAAAA"
+			"AAAAAAAAAAAAAAAAAAAAAAAAAAAAAAAAAAAAAAAAAAAAAAAAAAAAAAAAAAAAAAAAAAAAAAAAAAAA"
+			"AAAAAAAAAAAAAAAAAAAAAAAAAAAAAAAAAAAAAAAAAAAAAAAAAAAAAAAAAAAAAAAAAAAAAAAAAAAA"
+			"AAAAAAAAAAAAAAAAAAAAAAAAAAAAAAAAAAAAAAAAAAAAAAAAAAAAAAAAAAAAAAAAAAAAAAAAAAAA"
+			"AAAAAAAAAAAAAAAAAAAAAAAAAAAAAAAAAAAAAAAAAAAAAAAAAAAAAAAAAAAAAAAAAAAAAAAAAAAA"
+			"AAAAAAAAAAAAAAAAAAAAAAAAAAAAAAAAAAAAAAAAAAAAAAAAAAAAAAAAAAAAAAAAAAAAAAAAAAAA"
+			"AAAAAAAAAAAAAAAAAAAAAAAAAAAAAAAAAAAAAAAAAAAAAAAAAAAAAAAAAAAAAAAAAAAAAAAAAAAA"
 			"AAAAAAAAAAAAAAAAAAAAAAAAAAAAAAAAAAAAAAAAAAAAAAAAAAAAAAAAAAAAAA=="
 		)
@@
 	)
 	(symbol
-		(lib_id "PCM_LED_AKL:LED_1.8mm_SMD_Red")
+		(lib_id "all-comps:LED_1.8mm_SMD_Red")
 		(at 204.47 88.9 270)
 		(unit 1)
@@
 	)
 	(symbol
-		(lib_id "PCM_4ms_Capacitor:1uF_0603_25V")
+		(lib_id "all-comps:1uF_0603_25V")
 		(at 270.51 54.61 0)
 		(unit 1)
@@
 	)
 	(symbol
-		(lib_id "PCM_4ms_Resistor:10k_0402")
+		(lib_id "all-comps:10k_0402")
 		(at 361.95 116.84 0)
 		(unit 1)
@@
 	)
 	(symbol
-		(lib_id "PCM_4ms_Resistor:10k_0402")
+		(lib_id "all-comps:10k_0402")
 		(at 104.14 38.1 0)
 		(unit 1)
@@
 	)
 	(symbol
-		(lib_id "PCM_4ms_Capacitor:1uF_0603_25V")
+		(lib_id "all-comps:1uF_0603_25V")
 		(at 213.36 49.53 0)
 		(unit 1)
@@
 	)
 	(symbol
-		(lib_id "PCM_4ms_Resistor:10k_0402")
+		(lib_id "all-comps:10k_0402")
 		(at 144.78 49.53 0)
 		(unit 1)
@@
 	)
 	(symbol
-		(lib_id "PCM_4ms_Capacitor:1uF_0603_25V")
+		(lib_id "all-comps:1uF_0603_25V")
 		(at 255.27 33.02 0)
 		(unit 1)
@@
 	)
 	(symbol
-		(lib_id "PCM_4ms_Resistor:10k_0402")
+		(lib_id "all-comps:10k_0402")
 		(at 50.8 36.83 270)
 		(unit 1)
@@
 	)
 	(symbol
-		(lib_id "PCM_SL_Pin_Headers:PINHD_1x10_Female")
+		(lib_id "all-comps:PINHD_1x10_Female")
 		(at 328.93 74.93 180)
 		(unit 1)
@@
 	)
 	(symbol
-		(lib_id "PCM_4ms_Resistor:10k_0402")
+		(lib_id "all-comps:10k_0402")
 		(at 199.39 121.92 180)
 		(unit 1)
@@
 	)
 	(symbol
-		(lib_id "PCM_4ms_Capacitor:1uF_0603_25V")
+		(lib_id "all-comps:1uF_0603_25V")
 		(at 137.16 40.64 0)
 		(unit 1)
@@
 	)
 	(symbol
-		(lib_id "PCM_Diode_TVS_AKL:USBLC6-2SC6")
+		(lib_id "all-comps:USBLC6-2SC6")
 		(at 64.77 72.39 270)
 		(unit 1)
@@
 	)
 	(symbol
-		(lib_id "PCM_4ms_Resistor:10k_0402")
+		(lib_id "all-comps:10k_0402")
 		(at 351.79 127 90)
 		(unit 1)
@@
 	)
 	(symbol
-		(lib_id "PCM_4ms_Capacitor:1uF_0603_25V")
+		(lib_id "all-comps:1uF_0603_25V")
 		(at 82.55 44.45 180)
 		(unit 1)
@@
 	)
 	(symbol
-		(lib_id "PCM_4ms_Capacitor:1uF_0603_25V")
+		(lib_id "all-comps:1uF_0603_25V")
 		(at 264.16 33.02 0)
 		(unit 1)
@@
 	)
 	(symbol
-		(lib_id "PCM_SL_Pin_Headers:PINHD_1x10_Female")
+		(lib_id "all-comps:PINHD_1x10_Female")
 		(at 365.76 73.66 0)
 		(unit 1)
@@
 	)
 	(symbol
-		(lib_id "Diode:MBR1020VL")
+		(lib_id "all-comps:MBR1020VL")
 		(at 91.44 33.02 180)
 		(unit 1)
@@
 	)
 	(symbol
-		(lib_id "PCM_4ms_Capacitor:1uF_0603_25V")
+		(lib_id "all-comps:1uF_0603_25V")
 		(at 361.95 134.62 0)
 		(unit 1)
@@
 	)
 	(symbol
-		(lib_id "Device:Fuse_Small")
+		(lib_id "all-comps:Fuse_Small")
 		(at 76.2 33.02 0)
 		(unit 1)
@@
 	)
 	(symbol
-		(lib_id "PCM_4ms_Resistor:10k_0402")
+		(lib_id "all-comps:10k_0402")
 		(at 204.47 97.79 0)
 		(unit 1)
@@
 	)
 	(symbol
-		(lib_id "PCM_4ms_Resistor:10k_0402")
+		(lib_id "all-comps:10k_0402")
 		(at 203.2 121.92 0)
 		(unit 1)
@@
 	)
 	(symbol
-		(lib_id "MCU_Microchip_SAMD:ATSAMD21E16B-M")
+		(lib_id "all-comps:ATSAMD21E16B-M")
 		(at 246.38 100.33 0)
 		(unit 1)
@@
 	)
 	(symbol
-		(lib_id "Connector:USB_C_Receptacle_USB2.0_16P")
+		(lib_id "all-comps:USB_C_Receptacle_USB2.0_16P")
 		(at 29.21 44.45 0)
 		(unit 1)
@@
 	)
 	(symbol
-		(lib_id "PCM_Voltage_Regulator_AKL:AP2112K-3.3TRG1")
+		(lib_id "all-comps:AP2112K-3.3TRG1")
 		(at 123.19 35.56 0)
 		(unit 1)
@@
 	)
 	(symbol
-		(lib_id "PCM_SL_Devices:Push_Button")
+		(lib_id "all-comps:Push_Button")
 		(at 341.63 134.62 90)
 		(unit 1)
@@
 	)
 	(symbol
-		(lib_id "PCM_4ms_Capacitor:1uF_0603_25V")
+		(lib_id "all-comps:1uF_0603_25V")
 		(at 99.06 44.45 0)
 		(unit 1)
@@
 	)
 	(symbol
-		(lib_id "PCM_4ms_Capacitor:1uF_0603_25V")
+		(lib_id "all-comps:1uF_0603_25V")
 		(at 283.21 54.61 180)
 		(unit 1)
@@
 	)
 	(symbol
-		(lib_id "PCM_SL_Pin_Headers:PINHD_1x5_Male")
+		(lib_id "all-comps:PINHD_1x5_Male")
 		(at 363.22 35.56 90)
 		(unit 1)
@@
 	)
 	(symbol
-		(lib_id "PCM_4ms_Capacitor:1uF_0603_25V")
+		(lib_id "all-comps:1uF_0603_25V")
 		(at 82.55 78.74 0)
 		(unit 1)
@@
 	)
 	(symbol
-		(lib_id "EE_RESISTORS:0402WGF1001TCE")
+		(lib_id "all-comps:0402WGF1001TCE")
 		(at 345.44 40.64 0)
 		(unit 1)
@@
 	)
 	(symbol
-		(lib_id "PCM_LED_AKL:LED_1.8mm_SMD_Red")
+		(lib_id "all-comps:LED_1.8mm_SMD_Red")
 		(at 144.78 39.37 270)
 		(unit 1)
@@
 	)
 	(symbol
-		(lib_id "PCM_4ms_Resistor:10k_0402")
+		(lib_id "all-comps:10k_0402")
 		(at 50.8 34.29 90)
 		(unit 1)
@@
 	)
 	(symbol
-		(lib_id "PCM_4ms_Capacitor:1uF_0603_25V")
+		(lib_id "all-comps:1uF_0603_25V")
 		(at 219.71 49.53 180)
 		(unit 1)
